Commit message: カメラと LiDAR の位置の差の補正: 距離もカメラから前方の距離にし、方位をピンホールの式に。URDF の laser / camera_link を CAD の位置に
Co-Authored-By: Devin AI <158243242+devin-ai-integration[bot]@users.noreply.github.com>

File: src/ai_car_description/urdf/ai_car.xacro (robot description, xacro)
@@ -13,4 +13,12 @@
   <xacro:property name="wheel_y"      value="${base_width/2 + wheel_width/2}"/>
   <xacro:property name="wheel_z"      value="0.0"/>
+  <!-- センサーの取り付け位置（battery_lidar_mount.scad の CAD 値）。
+       base_link の原点は天板の中心（前後・左右）、車軸の高さ。x: 前、y: 左、z: 上 -->
+  <xacro:property name="laser_x" value="0.043"/>   <!-- LiDAR の回転中心: 天板の中心から前 43 mm・左 8 mm -->
+  <xacro:property name="laser_y" value="0.008"/>
+  <xacro:property name="laser_h" value="0.175"/>   <!-- 光の高さ（床から）。取付面 162 mm + ヘッド内の発光部（推定） -->
+  <xacro:property name="camera_x" value="0.096"/>  <!-- カメラのレンズ: LiDAR から前 53 mm・右 44 mm -->
+  <xacro:property name="camera_y" value="-0.036"/>
+  <xacro:property name="camera_h" value="0.128"/>  <!-- レンズの高さ（床から） -->
   <material name="body_gray">
     <color rgba="0.3 0.3 0.35 1.0"/>
@@ -115,5 +123,5 @@
     <parent link="base_link"/>
     <child link="laser"/>
-    <origin xyz="0.0 0.0 ${base_height/2 + 0.0205}" rpy="0 0 0"/>
+    <origin xyz="${laser_x} ${laser_y} ${laser_h - wheel_radius}" rpy="0 0 0"/>
   </joint>
   <!-- カメラ: Raspberry Pi Camera Module v3 -->
@@ -137,5 +145,5 @@
     <parent link="base_link"/>
     <child link="camera_link"/>
-    <origin xyz="${base_length/2} 0 ${base_height/2}" rpy="0 0 0"/>
+    <origin xyz="${camera_x} ${camera_y} ${camera_h - wheel_radius}" rpy="0 0 0"/>
   </joint>
   <!-- 光学座標系 (REP-103: z前方, x右, y下) -->

Commit message: LiDAR の前方をカメラの光軸に合わせる「前方合わせ」を追加（固定角度なし、保存して起動時に反映）
Co-Authored-By: Devin AI <158243242+devin-ai-integration[bot]@users.noreply.github.com>

File: src/ai_car_description/urdf/ai_car.xacro (robot description, xacro)
@@ -17,5 +17,7 @@
   <xacro:property name="laser_x" value="0.043"/>   <!-- LiDAR の回転中心: 天板の中心から前 43 mm・左 8 mm -->
   <xacro:property name="laser_y" value="0.008"/>
-  <xacro:property name="laser_h" value="0.175"/>   <!-- 光の高さ（床から）。取付面 162 mm + ヘッド内の発光部（推定） -->
+  <xacro:property name="laser_h" value="0.175"/>
+  <!-- LiDAR の 0° と車体前方（カメラの光軸）のずれ [rad]。slam.launch.py が前方合わせの値を渡す -->
+  <xacro:arg name="laser_yaw" default="0.0"/>   <!-- 光の高さ（床から）。取付面 162 mm + ヘッド内の発光部（推定） -->
   <xacro:property name="camera_x" value="0.096"/>  <!-- カメラのレンズ: LiDAR から前 53 mm・右 44 mm -->
   <xacro:property name="camera_y" value="-0.036"/>
@@ -123,5 +125,5 @@
     <parent link="base_link"/>
     <child link="laser"/>
-    <origin xyz="${laser_x} ${laser_y} ${laser_h - wheel_radius}" rpy="0 0 0"/>
+    <origin xyz="${laser_x} ${laser_y} ${laser_h - wheel_radius}" rpy="0 0 $(arg laser_yaw)"/>
   </joint>
   <!-- カメラ: Raspberry Pi Camera Module v3 -->

Commit message: LiDAR の前方を実測値 -1.7° で前方カメラの正面に固定し、前方合わせボタンを削除。表示範囲を 3 m に固定
Co-Authored-By: Devin AI <158243242+devin-ai-integration[bot]@users.noreply.github.com>

File: src/ai_car_description/urdf/ai_car.xacro (robot description, xacro)
@@ -17,7 +17,6 @@
   <xacro:property name="laser_x" value="0.043"/>   <!-- LiDAR の回転中心: 天板の中心から前 43 mm・左 8 mm -->
   <xacro:property name="laser_y" value="0.008"/>
-  <xacro:property name="laser_h" value="0.175"/>
-  <!-- LiDAR の 0° と車体前方（カメラの光軸）のずれ [rad]。slam.launch.py が前方合わせの値を渡す -->
-  <xacro:arg name="laser_yaw" default="0.0"/>   <!-- 光の高さ（床から）。取付面 162 mm + ヘッド内の発光部（推定） -->
+  <xacro:property name="laser_yaw_deg" value="-1.7"/>  <!-- 前方カメラの正面に合わせた LiDAR の向き（dashboard.yaml の scan_angle_offset_deg と同じ） -->
+  <xacro:property name="laser_h" value="0.175"/>   <!-- 光の高さ（床から）。取付面 162 mm + ヘッド内の発光部（推定） -->
   <xacro:property name="camera_x" value="0.096"/>  <!-- カメラのレンズ: LiDAR から前 53 mm・右 44 mm -->
   <xacro:property name="camera_y" value="-0.036"/>
@@ -125,5 +124,5 @@
     <parent link="base_link"/>
     <child link="laser"/>
-    <origin xyz="${laser_x} ${laser_y} ${laser_h - wheel_radius}" rpy="0 0 $(arg laser_yaw)"/>
+    <origin xyz="${laser_x} ${laser_y} ${laser_h - wheel_radius}" rpy="0 0 ${radians(laser_yaw_deg)}"/>
   </joint>
   <!-- カメラ: Raspberry Pi Camera Module v3 -->

Commit message: 3D プリント部品: Pi カメラと液晶をなくし、2 眼カメラの受けと LiDAR の下の IMU の台を追加
Co-Authored-By: Devin AI <158243242+devin-ai-integration[bot]@users.noreply.github.com>

File: src/ai_car_description/urdf/ai_car.xacro (robot description, xacro)
@@ -19,7 +19,10 @@
   <xacro:property name="laser_yaw_deg" value="-1.7"/>  <!-- 前方カメラの正面に合わせた LiDAR の向き（dashboard.yaml の scan_angle_offset_deg と同じ） -->
   <xacro:property name="laser_h" value="0.175"/>   <!-- 光の高さ（床から）。取付面 162 mm + ヘッド内の発光部（推定） -->
-  <xacro:property name="camera_x" value="0.096"/>  <!-- カメラのレンズ: LiDAR から前 53 mm・右 44 mm -->
-  <xacro:property name="camera_y" value="-0.036"/>
-  <xacro:property name="camera_h" value="0.128"/>  <!-- レンズの高さ（床から） -->
+  <xacro:property name="camera_x" value="0.103"/>  <!-- 2 眼カメラの左目のレンズの先: LiDAR から前 60 mm・左 30 mm -->
+  <xacro:property name="camera_y" value="0.038"/>
+  <xacro:property name="camera_h" value="0.125"/>  <!-- レンズの高さ（床から） -->
+  <xacro:property name="imu_x" value="0.045"/>     <!-- IMU の基板の中心: ふたの上、LiDAR のヘッドの下（天板の中心から前 45 mm・右 13 mm） -->
+  <xacro:property name="imu_y" value="-0.013"/>
+  <xacro:property name="imu_h" value="0.140"/>     <!-- 基板の高さ（床から） -->
   <material name="body_gray">
     <color rgba="0.3 0.3 0.35 1.0"/>
@@ -126,10 +129,10 @@
     <origin xyz="${laser_x} ${laser_y} ${laser_h - wheel_radius}" rpy="0 0 ${radians(laser_yaw_deg)}"/>
   </joint>
-  <!-- カメラ: Raspberry Pi Camera Module v3 -->
+  <!-- カメラ: USB 2 眼カメラ（3D USB Camera）の左目 -->
   <link name="camera_link">
     <visual>
       <origin xyz="0 0 0" rpy="0 0 0"/>
       <geometry>
-        <box size="0.01 0.025 0.025"/>
+        <box size="0.01 0.08 0.017"/>
       </geometry>
       <material name="sensor_green"/>
@@ -138,8 +141,8 @@
       <origin xyz="0 0 0" rpy="0 0 0"/>
       <geometry>
-        <box size="0.01 0.025 0.025"/>
+        <box size="0.01 0.08 0.017"/>
       </geometry>
     </collision>
-    <xacro:box_inertia m="0.01" x="0.01" y="0.025" z="0.025"/>
+    <xacro:box_inertia m="0.045" x="0.01" y="0.08" z="0.017"/>
   </link>
   <joint name="camera_joint" type="fixed">
@@ -169,5 +172,5 @@
     <parent link="base_link"/>
     <child link="imu_link"/>
-    <origin xyz="-0.05 0 ${base_height/2}" rpy="0 0 0"/>
+    <origin xyz="${imu_x} ${imu_y} ${imu_h - wheel_radius}" rpy="0 0 0"/>
   </joint>
 </robot>

Commit message: 2 眼カメラを実測に合わせ、USB 端子を上にして四隅の M2 で板に留める形に変更。カバーの窓をレンズごとに分ける
Co-Authored-By: Devin AI <158243242+devin-ai-integration[bot]@users.noreply.github.com>

File: src/ai_car_description/urdf/ai_car.xacro (robot description, xacro)
@@ -19,7 +19,7 @@
   <xacro:property name="laser_yaw_deg" value="-1.7"/>  <!-- 前方カメラの正面に合わせた LiDAR の向き（dashboard.yaml の scan_angle_offset_deg と同じ） -->
   <xacro:property name="laser_h" value="0.175"/>   <!-- 光の高さ（床から）。取付面 162 mm + ヘッド内の発光部（推定） -->
-  <xacro:property name="camera_x" value="0.103"/>  <!-- 2 眼カメラの左目のレンズの先: LiDAR から前 60 mm・左 30 mm -->
+  <xacro:property name="camera_x" value="0.122"/>  <!-- 2 眼カメラの左目のレンズの先: LiDAR から前 79 mm・左 30 mm -->
   <xacro:property name="camera_y" value="0.038"/>
-  <xacro:property name="camera_h" value="0.125"/>  <!-- レンズの高さ（床から） -->
+  <xacro:property name="camera_h" value="0.112"/>  <!-- レンズの高さ（床から） -->
   <xacro:property name="imu_x" value="0.045"/>     <!-- IMU の基板の中心: ふたの上、LiDAR のヘッドの下（天板の中心から前 45 mm・右 13 mm） -->
   <xacro:property name="imu_y" value="-0.013"/>

Commit message: 前方カメラを Camera Module 3 Wide（camera_ros）に戻す
Co-Authored-By: Devin AI <158243242+devin-ai-integration[bot]@users.noreply.github.com>

File: src/ai_car_description/urdf/ai_car.xacro (robot description, xacro)
@@ -19,6 +19,6 @@
   <xacro:property name="laser_yaw_deg" value="-1.7"/>  <!-- 前方カメラの正面に合わせた LiDAR の向き（dashboard.yaml の scan_angle_offset_deg と同じ） -->
   <xacro:property name="laser_h" value="0.175"/>   <!-- 光の高さ（床から）。取付面 162 mm + ヘッド内の発光部（推定） -->
-  <xacro:property name="camera_x" value="0.122"/>  <!-- 2 眼カメラの左目のレンズの先: LiDAR から前 79 mm・左 30 mm -->
-  <xacro:property name="camera_y" value="0.038"/>
+  <xacro:property name="camera_x" value="0.106"/>  <!-- Camera Module 3 Wide のレンズの先: LiDAR の回転中心の真ん前 63 mm -->
+  <xacro:property name="camera_y" value="0.008"/>
   <xacro:property name="camera_h" value="0.112"/>  <!-- レンズの高さ（床から） -->
   <xacro:property name="imu_x" value="0.045"/>     <!-- IMU の基板の中心: ふたの上、LiDAR のヘッドの下（天板の中心から前 45 mm・右 13 mm） -->
@@ -129,10 +129,10 @@
     <origin xyz="${laser_x} ${laser_y} ${laser_h - wheel_radius}" rpy="0 0 ${radians(laser_yaw_deg)}"/>
   </joint>
-  <!-- カメラ: USB 2 眼カメラ（3D USB Camera）の左目 -->
+  <!-- カメラ: Camera Module 3 Wide（IMX708） -->
   <link name="camera_link">
     <visual>
       <origin xyz="0 0 0" rpy="0 0 0"/>
       <geometry>
-        <box size="0.01 0.08 0.017"/>
+        <box size="0.01 0.025 0.024"/>
       </geometry>
       <material name="sensor_green"/>
@@ -141,8 +141,8 @@
       <origin xyz="0 0 0" rpy="0 0 0"/>
       <geometry>
-        <box size="0.01 0.08 0.017"/>
+        <box size="0.01 0.025 0.024"/>
       </geometry>
     </collision>
-    <xacro:box_inertia m="0.045" x="0.01" y="0.08" z="0.017"/>
+    <xacro:box_inertia m="0.004" x="0.01" y="0.025" z="0.024"/>
   </link>
   <joint name="camera_joint" type="fixed">

Commit message: カメラの位置を実物に合わせる（端子を下にして付けているので、レンズの中心を天板から 28.1 mm に）
Co-Authored-By: Devin AI <158243242+devin-ai-integration[bot]@users.noreply.github.com>

File: src/ai_car_description/urdf/ai_car.xacro (robot description, xacro)
@@ -21,5 +21,5 @@
   <xacro:property name="camera_x" value="0.106"/>  <!-- Camera Module 3 Wide のレンズの先: LiDAR の回転中心の真ん前 63 mm -->
   <xacro:property name="camera_y" value="0.008"/>
-  <xacro:property name="camera_h" value="0.112"/>  <!-- レンズの高さ（床から） -->
+  <xacro:property name="camera_h" value="0.100"/>  <!-- レンズの高さ（床から。天板の上 28.1 mm） -->
   <xacro:property name="imu_x" value="0.045"/>     <!-- IMU の基板の中心: ふたの上、LiDAR のヘッドの下（天板の中心から前 45 mm・右 13 mm） -->
   <xacro:property name="imu_y" value="-0.013"/>
